File: N_5412K.sch (EAGLE design)
At the start: 64 parts

Commit message: Updating per what was wired in the hangar today
Parts:
- renumbered U$4 to PFD, U$5 to MFD
Connections:
- net AUX_GEA24 renamed AUX_GEA24_YR
- net AUX_PFD renamed AUX_PFD_YR
- net GND_GMC307_15 renamed GND_GMC307_GND2
- net GND_GMC307_5 renamed GND_GMC307_GND1
- net VPX_GEA_24 renamed VPX_GEA_24_R
- removed net AUX_GSU_25_1: AUX_FUSEBLOCK.9, GSU25_PRIMARY.AIRCRAFT_POWER2
- removed net B$7: PITCH.CAN-H, PITCH.CAN-L
- removed net CAN_HI: GAD29.J291_1, GMA-245.J2401_36, MFD.CAN_BUS_HI, PFD.CAN_BUS_HI, YAW.CAN-H
- removed net CAN_LO: GAD29.J291_2, GMA-245.J2401_37, MFD.CAN_BUS_LO, PFD.CAN_BUS_LO, YAW.CAN-L
- removed net GEA23_SHUNT_HI: GEA24.J243_37
- removed net GEA24_SHUNT_LO: GEA24.J243_36, U$10.2
- removed net GND_PFD1: PFD.PWR_GND1
- removed net GND_PFD2: PFD.PWR_GND_2
- new net AUX_GSU_25_1_YR: AUX_FUSEBLOCK.9, GSU25_PRIMARY.8_AIRCRAFT_POWER2
- new net CAN_BUS_PITCH_SERVO: GAD29.J291_1, GAD29.J291_2, GEA24.CAN_HI_1, GEA24.CAN_LO_2, GMA-245.J2401_36, GMA-245.J2401_37, GSU25_BACKUP.1_CAN_H, GSU25_BACKUP.2_CAN_L, GSU25_PRIMARY.1_CAN_H, GSU25_PRIMARY.2_CAN_L, GTR-20.J2001_6, GTR-20.J2001_7, MFD.1_CAN_BUS_HI, MFD.2_CAN_BUS_LO, PFD.1_CAN_BUS_HI, PFD.2_CAN_BUS_LO, PITCH.CAN-H, PITCH.CAN-L, YAW.CAN-H, YAW.CAN-L
- new net GND_GEA24_1_B: GEA24.J241_6
- new net GND_GEA24_2_B: GEA24.J241_9
- new net GND_PFD1_B: PFD.15_PWR_GND1
- new net GND_PFD2_B: PFD.16_PWR_GND_2
- new net N$14: GTN650.P1001_45, PFD.34_SIGNAL_GROUND2
- new net N$24: AUX_FUSEBLOCK.IN_1, AUX_FUSEBLOCK.IN_2, U$10.I
- new net PFD_RS232[4]_W: GSU25_PRIMARY.4_RS232_RX1, PFD.5_RS-232-RX
- new net PFD_RS232[5]_WB: GSU25_PRIMARY.5_RS232_TX1, PFD.4_RS_232_TX
- new net RS232_W: GEA24.RS232_TX_5, PFD.23_RS-232-IN4
- new net RS232_WB: GEA24.RS232_RX_4, PFD.40_RS-232-OUT4
- new net SEN_AUX_VOLTAGE: AUX_FUSEBLOCK.11, GEA24.J244_28
- new net SEN_SHUNT2_HI_W: GEA24.J243_35, U$10.2
- new net SEN_SHUNT2_LO_WB: GEA24.J243_34, U$10.1
- net ADHARS_2: now also GSU25_BACKUP.UNIT_ID1_GND_4, GSU25_BACKUP.UNIT_ID_5; no longer GSU25_BACKUP.UNIT_ID1, GSU25_BACKUP.UNIT_ID1_GND
- net B$1: no longer GSU25_PRIMARY.OAT_HIGH, GSU25_PRIMARY.OAT_LOW, GSU25_PRIMARY.OAT_PWR
- net BATT_AUX: now also U$10.O; no longer AUX_FUSEBLOCK.IN_1, AUX_FUSEBLOCK.IN_2
- net GMC_307_IN1_WHT/BLU: now also MFD.48_RS-232-OUT1; no longer MFD.RS-232-OUT1
- net GMC_307_OUT1_WHT: now also MFD.47_RS-232-IN1; no longer MFD.RS-232-IN1
- net GMU_22_485: now also GSU25_PRIMARY.RS485_RXA_12, GSU25_PRIMARY.RS485_RXB_13; no longer GSU25_PRIMARY.RS485_RXA, GSU25_PRIMARY.RS485_RXB
- net GMU_22_PWR: now also GSU25_PRIMARY.12V_MAG_PWR_6, GSU25_PRIMARY.MAG_GND_7; no longer GSU25_PRIMARY.12V_MAG_PWR, GSU25_PRIMARY.MAG_GND
- net GND: no longer GEA24.J241_6, GEA24.J241_9
- net GND_GSU25_BACK_1: now also GSU25_BACKUP.6_GND1, GSU25_BACKUP.9_GND2; no longer GSU25_BACKUP.GND1, GSU25_BACKUP.GND2
- net GND_GSU25_PRI_1: now also GSU25_PRIMARY.6_GND1; no longer GSU25_PRIMARY.GND1
- net GND_GSU25_PRI_2: now also GSU25_PRIMARY.9_GND2; no longer GSU25_PRIMARY.GND2
- net GND_MFD1: now also MFD.15_PWR_GND1; no longer MFD.PWR_GND1
- net GND_MFD2: now also MFD.16_PWR_GND_2; no longer MFD.PWR_GND_2
- net MFD_51RTX: now also MFD.14_RS-232-IN2; no longer MFD.RS-232-IN2
- net N$11: now also GTN650.P1001_26, PFD.RS-232-OUT2; no longer GSU25_BACKUP.CAN_H, GSU25_PRIMARY.CAN_H
- net N$13: now also PFD.10_CDU_SYSTEM_ID_PRG_1; no longer PFD.CDU_SYSTEM_ID_PRG_1
- net N$15: now also MFD.34_SIGNAL_GROUND2; no longer MFD.SIGNAL_GROUND2
- net N$18: now also GTN650.P1001_7, PFD.14_RS-232-IN2; no longer GEA24.J244_28
- net N$2: now also GTN650.P1001_46, PFD.37_SIGNAL_GROUND5; no longer GSU25_BACKUP.CAN_L, GSU25_PRIMARY.CAN_L
- net N$21: now also PFD.35_SIGNAL_GROUND3; no longer PFD.SIGNAL_GROUND3
- net N$4: no longer U$10.O
- net N$6: no longer U$10.I
- net OAT: now also GSU25_PRIMARY.OAT_HIGH_2, GSU25_PRIMARY.OAT_LOW_3, GSU25_PRIMARY.OAT_PWR_1
- net PFD_51R_RX: now also PFD.13_RS-232-OUT3; no longer PFD.RS-232-OUT3
- net PFD_RS232_RX1: now also GTN650.P1001_8, PFD.47_RS-232-IN1; no longer PFD.RS-232-IN1
- net PFD_RS232_TX1: now also GTN650.P1001_27, PFD.48_RS-232-OUT1; no longer PFD.RS-232-OUT1
- net REVERISIONARY_MODE: now also MFD.25_CDU_SYSTEM_ID_PRG_3; no longer MFD.CDU_SYSTEM_ID_PRG_3
- net SERIAL_GND_WHT/ORN: now also MFD.35_SIGNAL_GROUND3; no longer MFD.SIGNAL_GROUND3
- net SERIAL_RX_WHT/BLU: now also MFD.13_RS-232-OUT3; no longer MFD.RS-232-OUT3
- net VPX_ALT1: now also 1224.AUX, 1224.SENSE
- net VPX_GSU_25_1: now also GSU25_PRIMARY.7_AIRCRAFT_POWER1; no longer GSU25_PRIMARY.AIRCRAFT_POWER1
- net VPX_GSU_25_2: now also GSU25_BACKUP.7_AIRCRAFT_POWER1; no longer GSU25_BACKUP.AIRCRAFT_POWER1
Other:
- moved on the sheet: GTN650, MANIFOLD, SW_AUTOPILOT, SW_BOOST, U$10, U$9

Commit message: Updating per what was wired in the hangar today
Parts:
- added U$4: SHIELD, EAA:SHIELD
Connections:
- removed net GMU_22_485: GSU25_PRIMARY.RS485_RXA_12, GSU25_PRIMARY.RS485_RXB_13
- removed net GMU_22_485_SHIELD: U$11.SIGNAL_GND2
- removed net GMU_22_485_W: U$11.RS485_OUTA
- removed net GMU_22_485_WB: U$11.RS485_OUTB
- removed net GMU_22_PWR: GSU25_PRIMARY.12V_MAG_PWR_6, GSU25_PRIMARY.MAG_GND_7
- removed net GMU_22_PWR_SHIELD: U$11.SIGNAL_GND1
- removed net GMU_22_PWR_W: U$11.RS232_IN
- removed net GMU_22_PWR_WB: U$11.GND
- removed net GMU_22_PWR_WO: U$11.12V_PWR
- removed net MFD_51RTX: GDL51R.RS232_TX1, MFD.14_RS-232-IN2
- removed net MFD_51R_RX: GDL51R.RS232_RX1, MFD.RS-232-OUT2
- removed net N$11: GTN650.P1001_26, PFD.RS-232-OUT2
- removed net N$14: GTN650.P1001_45, PFD.34_SIGNAL_GROUND2
- removed net N$15: GDL51R.SIGNAL_GND1, MFD.34_SIGNAL_GROUND2
- removed net N$18: GTN650.P1001_7, PFD.14_RS-232-IN2
- removed net N$2: GTN650.P1001_46, PFD.37_SIGNAL_GROUND5
- removed net N$21: GDL51R.SIGNAL_GND2, PFD.35_SIGNAL_GROUND3
- removed net OAT: GSU25_PRIMARY.OAT_HIGH_2, GSU25_PRIMARY.OAT_LOW_3, GSU25_PRIMARY.OAT_PWR_1, GTP59.HIGH, GTP59.LOW, GTP59.PWR
- removed net PFD_51R_RX: GDL51R.RS232_RX2, PFD.13_RS-232-OUT3
- removed net PFD_51R_TX: GDL51R.RS232_TX2, PFD.RS-232-IN3
- removed net PFD_RS232[4]_W: GSU25_PRIMARY.4_RS232_RX1, PFD.5_RS-232-RX
- removed net PFD_RS232[5]_WB: GSU25_PRIMARY.5_RS232_TX1, PFD.4_RS_232_TX
- removed net PFD_RS232_RX1: GTN650.P1001_8, PFD.47_RS-232-IN1
- removed net PFD_RS232_TX1: GTN650.P1001_27, PFD.48_RS-232-OUT1
- removed net SERIAL_GND_WHT/ORN: MFD.35_SIGNAL_GROUND3
- removed net SERIAL_RX_WHT/BLU: MFD.13_RS-232-OUT3
- removed net SERIAL_TX_WHT: MFD.RS-232-IN3
- new net 441_2_WB: U$11.2_RS485_OUTB
- new net 441_4_W: U$11.4_RS485_OUTA
- new net 441_6_WB: U$11.6_GND
- new net 441_8_W: U$11.8_RS232_IN
- new net 441_9_WO: U$11.9_12V_PWR
- new net 4601_4_W: PFD.4_RS_232_TX
- new net 4601_5_WB: PFD.5_RS-232-RX
- new net 4602_14_W: MFD.14_RS-232-IN2
- new net 4602_30_WO: MFD.30_RS-232-OUT2
- new net 4602_34_WB: MFD.34_SIGNAL_GROUND2
- new net CAN_HI: GAD29.J291_1, GMA-245.J2401_36, MFD.1_CAN_BUS_HI
- new net CAN_HI_W: GEA24.CAN_HI_1, GSU25_BACKUP.1_CAN_H, GSU25_PRIMARY.1_CAN_H, GTR-20.J2001_7, PFD.1_CAN_BUS_HI
- new net CAN_LO: GAD29.J291_2, GMA-245.J2401_37, MFD.2_CAN_BUS_LO
- new net CAN_LO_WB: GEA24.CAN_LO_2, GSU25_BACKUP.2_CAN_L, GSU25_PRIMARY.2_CAN_L, GTR-20.J2001_6, PFD.2_CAN_BUS_LO
- new net GDL51_11_WB: GDL51R.4
- new net GDL51_12_WB: GDL51R.12_SIGNAL_GND2
- new net GDL51_5_W: GDL51R.5_RS232_TX2
- new net GDL51_6_WO: GDL51R.6_RS232_RX2
- new net GDL51_7_W: GDL51R.7_RS232_TX1
- new net GDL51_8_WO: GDL51R.8_RS232_RX1
- new net GTN650_1001_26_WO: GTN650.P1001_26
- new net GTN650_1001_27_WO: GTN650.P1001_27
- new net GTN650_1001_45_WB: GTN650.P1001_45
- new net GTN650_1001_46_WB: GTN650.P1001_46
- new net GTN650_1001_7_W: GTN650.P1001_7
- new net GTN650_1001_8_W: GTN650.P1001_8
- new net HIGH_2: GSU25_PRIMARY.OAT_HIGH_2
- new net HIGH_2_WB: GTP59.HIGH
- new net J251_4_W: GSU25_PRIMARY.4_RS232_RX1
- new net J251_5_WB: GSU25_PRIMARY.5_RS232_TX1
- new net LOW_3: GSU25_PRIMARY.OAT_LOW_3
- new net LOW_3_WO: GTP59.LOW
- new net PFD_13_WO: PFD.13_RS-232-OUT3
- new net PFD_14_W: PFD.14_RS-232-IN2
- new net PFD_24_W: PFD.24_RS-232-IN5
- new net PFD_29_W: PFD.29_RS-232-IN3
- new net PFD_30_WO: PFD.30_RS-232-OUT2
- new net PFD_34_WB: PFD.34_SIGNAL_GROUND2
- new net PFD_35_WB: PFD.35_SIGNAL_GROUND3
- new net PFD_36_WB: PFD.36_SIGNAL_GROUND4
- new net PFD_37_WB: PFD.37_SIGNAL_GROUND5
- new net PFD_41_WO: PFD.41_RS-232-OUT5
- new net PFD_47_W: PFD.47_RS-232-IN1
- new net PFD_48_WO: PFD.48_RS-232-OUT1
- new net PWR_1: GSU25_PRIMARY.OAT_PWR_1
- new net PWR_1_WO: GTP59.PWR
- new net S: U$11.1_SIGNAL_GND1, U$11.3_SIGNAL_GND2, U$4.S
- net ACK_GPS_RX: no longer GTN650.P1001_5
- net CAN_BUS_PITCH_SERVO: no longer GAD29.J291_1, GAD29.J291_2, GEA24.CAN_HI_1, GEA24.CAN_LO_2, GMA-245.J2401_36, GMA-245.J2401_37, GSU25_BACKUP.1_CAN_H, GSU25_BACKUP.2_CAN_L, GSU25_PRIMARY.1_CAN_H, GSU25_PRIMARY.2_CAN_L, GTR-20.J2001_6, GTR-20.J2001_7, MFD.1_CAN_BUS_HI, MFD.2_CAN_BUS_LO, PFD.1_CAN_BUS_HI, PFD.2_CAN_BUS_LO
- net GAD29_ARINC_IN_1A: no longer GTN650.P1001_10
- net GAD29_ARNIC_IN_1B: no longer GTN650.P1001_29
- net GND_GDL_51: now also GDL51R.9_GND; no longer GDL51R.GND
- net VPX_GDL_51R: now also GDL51R.10_PWR; no longer GDL51R.PWR
Other:
- moved on the sheet: GDL51R, GTN650, U$11

Commit message: Adding phones
Parts:
- removed LANDING/TAXI, X-FEED: TL46YO, switch:TL46YO
- removed USB: (no value), switch-omron:31-XX
- added CO-PILOT_MIC, CO-PILOT_PHONE, PASSENGER1_MIC, PASSENGER1_PHONE, PASSENGER2_MIC, PASSENGER2_PHONE, PILOT_MIC, PILOT_PHONE: PG203J, con-hirschmann:PG203J
- added SW-XFEED, SW_NAV_C, SW_TRIM_DOWN, SW_TRIM_LEFT, SW_TRIM_RIGHT, SW_TRIM_UP: (no value), switch-omron:31-XX
- added SW_TAXI_LANDING_C: TL46YO, switch:TL46YO
- added U$5: CPC_28, EAA:CPC_28
- added USB_CHGR: WM16793-ND, EAA:WM16793-ND
- renumbered POS/STROBE to SW_STROBE_C, SW_AUTOPILOT to SW_AUTOPILOT_C, SW_PITOT to SW_PITOT_C
Connections:
- net GAD29_ARNIC_OUT_1A renamed GAD29_2_W
- net GAD29_ARNIC_OUT_1B renamed GAD29_2_WB
- removed net GAD29_ARINC_IN_1A: GAD29.J292_23
- removed net GAD29_ARNIC_IN_1B: GAD29.J292_11
- removed net N$7: GTN650.P1001_19
- removed net N$8: X-FEED.P
- new net CPM_S: U$5.L$28
- new net CPM_W: CO-PILOT_MIC.2, U$5.L$26
- new net CPM_WB: CO-PILOT_MIC.1, CO-PILOT_MIC.5, U$5.L$27
- new net CPP_S: U$5.L$25
- new net CPP_W: CO-PILOT_PHONE.5, U$5.L$22
- new net CPP_WB: CO-PILOT_PHONE.1, U$5.L$23
- new net CPP_WO: CO-PILOT_PHONE.2, U$5.L$24
- new net D_WR: SW_TRIM_DOWN.S
- new net GAD29_1_W: GAD29.J292_23, GTN650.P1001_9
- new net GAD29_1_WB: GAD29.J292_11, GTN650.P1001_29
- new net L_B: SW_TRIM_LEFT.S
- new net P1M_S: U$5.L$10
- new net P1M_W: PASSENGER1_MIC.2, U$5.L$8
- new net P1M_WB: PASSENGER1_MIC.1, U$5.L$9
- new net P2M_S: U$5.L$13
- new net P2M_W: PASSENGER2_MIC.2, U$5.L$11
- new net P2M_WB: PASSENGER2_MIC.1, U$5.L$12
- new net PASSP_S: U$5.L$7
- new net PASSP_W: PASSENGER1_PHONE.2, PASSENGER2_PHONE.2, U$5.L$4
- new net PASSP_WB: PASSENGER1_PHONE.1, PASSENGER2_PHONE.1, U$5.L$5
- new net PASSP_WO: PASSENGER1_PHONE.5, PASSENGER2_PHONE.5, U$5.L$6
- new net PM_S: U$5.L$21
- new net PM_W: PILOT_MIC.2, U$5.L$18
- new net PM_WB: PILOT_MIC.1, U$5.L$19
- new net PM_WO: PILOT_MIC.5, U$5.L$20
- new net PP_S: U$5.L$17
- new net PP_W: PILOT_PHONE.2, PILOT_PHONE.5, U$5.L$14
- new net PP_WB: PILOT_PHONE.1, U$5.L$15
- new net PP_WO: U$5.L$16
- new net R_WB: SW_TRIM_RIGHT.S
- new net SW_WIGWAG: SW_STROBE_C.S1, U$1.J2_11
- new net USB_GND_WB: U$5.L$2, USB_CHGR.P$4
- new net USB_POS_W: U$5.L$1, USB_CHGR.P$1
- new net USB_S: U$5.L$3
- new net U_R: SW_TRIM_UP.S
- net GND: now also SW-XFEED.P; no longer X-FEED.P1
- net N$23: now also GTN650.P1001_19
- net PFD_24_W: now also GTX45R.P3251_7
- net PFD_35_WB: now also GTX45R.P3251_50
- net PFD_41_WO: now also GTX45R.P3251_29
- net SW_LANDING: now also SW_TAXI_LANDING_C.S1; no longer LANDING/TAXI.S1
- net SW_NAV: now also SW_NAV_C.S; no longer SW_STROBE_C.S1
- net SW_TAXI: now also SW_TAXI_LANDING_C.S; no longer LANDING/TAXI.S
- net X-FEED_CONTACTOR: now also SW-XFEED.S; no longer X-FEED.S1
Other:
- moved on the sheet: GTN650

Commit message: Converting more twisted pairs to busses
Parts:
- removed BKR_IGN1: 5A, EAA:BREAKER
- removed IGN1: (no value), switch-omron:31-XX
- removed R2: (no value), rcl:R-US_0922/22
- removed SW_TAXI_LANDING_C: TL46YO, switch:TL46YO
- added SW_LT: TL46YO, switch:TL46YO
- added SW_TRIM_DOWN1, SW_TRIM_LEFT1, SW_TRIM_RIGHT1, SW_TRIM_UP1: (no value), switch-omron:31-XX
- added U$12: FORREST_OF_TABS, EAA:FORREST_OF_TABS
- added U$13: CPC_15, EAA:CPC_15
- U$4: value SHIELD -> G3X_CONFIG; device EAA:SHIELD -> EAA:G3X_CONFIG
Connections:
- net N$16 renamed VPX_SERIAL_WB
- net N$22 renamed VPX_SERIAL_WO
- net N$3 renamed VPX_SERIAL_W
- net RS232_W renamed GEA24_RS232_W
- net RS232_WB renamed GEA24_RS232_WB
- removed net AUTOPILOT_ROLL: ROLL.SERVO_PWR
- removed net AUX_BUS: R2.1
- removed net CWS/DISC: ROLL.CWS/DISC
- removed net GND_GMA245_11: GMA-245.2402_11
- removed net GND_KEYSWITCH: STARTER_SWITCH.GND
- removed net GND_SW_AVIONICS: AVIONICS.P, AVIONICS.P1
- removed net GND_SW_MASTER: MASTER.P, MASTER.P1
- removed net N$1: R2.2, U$1.J2_12
- removed net PFD_36_WB: PFD.36_SIGNAL_GROUND4
- removed net ROLL_RS232_RX: ROLL.RS232_RX/STRAP4
- removed net ROLL_RS232_TX: ROLL.RS232_TX/STRAP3
- removed net SW_IGN1: BKR_IGN1.0, IGN1.P
- removed net SYSTEM32_IGN1: IGN1.S
- removed net USB_S: U$5.L$3
- new net CPM_WO: CO-PILOT_MIC.5, U$5.L$28
- new net GMA245_29_W: GMA-245.J2401_29
- new net GMA245_43_WB: GMA-245.J2401_43
- new net GMA245_CPM_S: U$5.P$3
- new net GMA245_CPM_W: U$5.P$26
- new net GMA245_CPM_WB: GMA-245.J2402_32, GMA-245.J2402_34, U$5.P$27
- new net GMA245_CPM_WO: GMA-245.J2402_33, U$5.P$28
- new net GMA245_CPP_S: U$5.P$25
- new net GMA245_CPP_W: GMA-245.2402_3, U$5.P$22
- new net GMA245_CPP_WB: GMA-245.2402_2, U$5.P$23
- new net GMA245_CPP_WO: GMA-245.2402_4, U$5.P$24
- new net GMA245_E1_W: GDL51R.13_MUSIC_OUT_LEFT, GMA-245.J2402_23
- new net GMA245_E1_WB: GDL51R.14_MUSIC_OUT_COMMON, GMA-245.J2402_25
- new net GMA245_E1_WO: GDL51R.15_MUSIC_OUT_RIGHT, GMA-245.J2402_24
- new net GMA245_PAPH_S: U$5.P$7
- new net GMA245_PAPH_W: GMA-245.J2401_40, U$5.P$4
- new net GMA245_PAPH_WB: GMA-245.J2401_42, U$5.P$5
- new net GMA245_PAPH_WO: GMA-245.J2401_41, U$5.P$6
- new net GMA245_PLM_S: U$5.P$13
- new net GMA245_PLM_W: GMA-245.J2402_37, U$5.P$11
- new net GMA245_PLM_WB: GMA-245.J2402_38, U$5.P$12
- new net GMA245_PM_S: U$5.P$21
- new net GMA245_PM_W: GMA-245.J2401_33, U$5.P$18
- new net GMA245_PM_WB: GMA-245.J2401_35, U$5.P$19
- new net GMA245_PM_WO: GMA-245.J2401_34, U$5.P$20
- new net GMA245_PP_S: U$5.P$17
- new net GMA245_PP_W: GMA-245.J2402_16, U$5.P$14
- new net GMA245_PP_WB: GMA-245.2402_1, U$5.P$15
- new net GMA245_PP_WO: GMA-245.J2402_31, U$5.P$16
- new net GMA245_PRM_S: U$5.P$10
- new net GMA245_PRM_W: GMA-245.J2402_35, U$5.P$8
- new net GMA245_PRM_WB: GMA-245.J2402_36, U$5.P$9
- new net J252_12_W: GSU25_PRIMARY.RS485_RXA_12
- new net J252_13_WB: GSU25_PRIMARY.RS485_RXB_13
- new net J252_15_W: GSU25_PRIMARY.RS232_TX2_15
- new net J252_6_WO: GSU25_PRIMARY.12V_MAG_PWR_6
- new net J252_7_WBS: GSU25_PRIMARY.MAG_GND_7
- new net N$11: ROLL.CAN-TERM1, ROLL.CAN-TERM2
- new net N$14: ROLL.TRIM_OUT1, U$13.L$13
- new net N$15: ROLL.TRIM_OUT2, U$13.L$14
- new net N$16: PFD.33_CONFIG_MODULE_CLOCK, U$4.WHT
- new net N$18: ROLL.CWS/DISC, U$13.L$15
- new net N$19: ROLL.TRIM_IN2, U$13.L$12
- new net N$2: ROLL.SERVO_GND, U$13.L$9
- new net N$21: ROLL.TRIM_IN1, U$13.L$11
- new net N$22: PFD.49_CONFIG_MODULE_GROUND, U$4.BLK
- new net N$26: PFD.50_CONFIG_MODULE_DATA, U$4.YEL
- new net N$3: PFD.17_CONFIG_MODULE_PWR_OUT, U$4.RED
- new net N$7: ROLL.CAN-H, U$13.L$1
- new net N$8: ROLL.CAN-L, U$13.L$2
- new net PFD_18_WB: PFD.18_MONO_AUDIO_OUT_LO
- new net PFD_1_W: PFD.1_MONO_AUDIO_OUT_HI
- new net PFD_27_WB: PFD.27_SIGNAL_GROUND1
- new net RTRIM1_W/G: U$13.P$12
- new net RTRIM2_W/G: U$13.P$11
- new net VCC: U$13.L$3
- net BATT_MAIN: no longer BKR_IGN1.I
- net CAN_HI_W: now also U$13.P$1
- net CAN_LO_WB: now also U$13.P$2
- net CPM_S: now also U$5.L$3; no longer U$5.L$28
- net CPM_WB: no longer CO-PILOT_MIC.5
- net GND: now also AVIONICS.P, AVIONICS.P1, MASTER.P, MASTER.P1, SW-XFEED.S, U$12.GND2; no longer ROLL.SERVO_GND, SW-XFEED.P
- net GND_GEA24_1_B: now also U$12.P$20
- net GND_GEA24_2_B: now also U$12.P$10
- net GND_GMA245_10: now also GMA-245.2402_11
- net N$13: now also PFD.44_SIGNAL_GROUND6; no longer PFD.SIGNAL_GROUND1
- net N$4: now also ROLL.SERVO_PWR, U$13.L$10; no longer U$2.IN, U$6.I
- net N$6: now also U$2.IN, U$6.I
- net PFD_35_WB: no longer PFD.35_SIGNAL_GROUND3
- net REVERISIONARY_MODE: no longer MFD.25_CDU_SYSTEM_ID_PRG_3
- net S: no longer U$4.S
- net SW_ALT1: now also ALT_SEL.O; no longer ALT_SEL.S1
- net SW_ALT2: now also ALT_SEL.O1; no longer ALT_SEL.O
- net SW_LANDING: now also SW_LT.S1; no longer SW_TAXI_LANDING_C.S1
- net SW_TAXI: now also SW_LT.S; no longer SW_TAXI_LANDING_C.S
- net USB_GND_WB: no longer U$5.L$2
- net USB_POS_W: no longer U$5.L$1
- net VPX_MFD: no longer MFD.AIRCRAFT_POWER_2
- net X-FEED_CONTACTOR: now also SW-XFEED.P; no longer SW-XFEED.S
Other:
- moved on the sheet: ALT_SEL, AVIONICS, GMA-245, MASTER, ROLL, STARTER_SWITCH, SW-XFEED, SW_AUTOPILOT_C, SW_BOOST, SW_NAV_C, SW_PITOT_C, SW_STROBE_C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

Commit message: Adding more Garmin components, cleaning up the pins on existing ones
Parts:
- added ROLL_TRIM: RAYALLEN_T2, EAA:RAYALLEN_T2
Connections:
- net COM1_AUDIO_HI renamed C1A_W
- net COM1_MIC_HI renamed C1M_W
- net COM2_MIC_HI renamed C2M_W
- net COM2_MIC_KEY renamed C2M_WO
- net COM_MIC_KEY renamed C1M_WO
- net CWS_DISC renamed CWS_DISC_WB
- net GAD29_ARNIC_IN_2A renamed AV_W
- net GAD29_ARNIC_IN_2B renamed AV_WB
- net N$46 renamed EI1_W
- net N$47 renamed EI1_WB
- net STROBE_SYNC renamed SS_BLUE
- removed net B$1: PITCH.TRIM_IN1, PITCH.TRIM_IN2
- removed net B$2: PITCH.TRIM_OUT1, PITCH.TRIM_OUT2, PITCH_TRIM.MOTOR1, PITCH_TRIM.MOTOR2
- removed net B$3: PITCH_TRIM.WHITE_BLUE, PITCH_TRIM.WHITE_GREEN, PITCH_TRIM.WHITE_ORANGE
- removed net CAN_BUS_PITCH_SERVO: PITCH.CAN-H, PITCH.CAN-L, YAW.CAN-H, YAW.CAN-L
- removed net CAN_HI: GAD29.J291_1, GMA-245.J2401_36, MFD.1_CAN_BUS_HI
- removed net CAN_LO: GAD29.J291_2, GMA-245.J2401_37, MFD.2_CAN_BUS_LO
- removed net COM1_LO: GMA-245.J2401_10, GTN650.P1003_18, GTN650.P1003_20
- removed net COM2_AUDIO_HI: GMA-245.J2401_13, GTR-20.J2001_10
- removed net COM2_LO: GMA-245.J2401_14, GTR-20.J2001_29, GTR-20.J2001_36
- removed net N$17: GTN650.P1002_24, GTX45R.P3252_1
- removed net N$45: GTN650.P1002_23, GTX45R.P3252_6
- removed net PFD_35_WB: GTX45R.P3251_50
- removed net TAIL_STROBE: POSI-STROBE.GND, POSI-STROBE.POSITION, POSI-STROBE.STROBE
- new net A1_W: GMA-245.J2401_31, GTN650.P1001_4
- new net A1_WB: GMA-245.J2401_32, GTN650.P1001_23
- new net C1A_WB: GMA-245.J2401_10, GTN650.P1003_18
- new net C1M_WB: GTN650.P1003_20
- new net C2A_W: GMA-245.J2401_13, GTR-20.J2001_29
- new net C2A_WB: GTR-20.J2001_10
- new net C2M_WB: GMA-245.J2401_14, GTR-20.J2001_36
- new net E01_WB: GTN650.P1002_24, GTX45R.P3252_1, GTX45R.P3252_6
- new net EO1_W: GTN650.P1002_23
- new net N$1: AUX_FUSEBLOCK.1
- new net N$29: GTX45R.P3251_45
- new net N$30: GTX45R.P3251_44
- new net N$31: GTX45R.P3251_24
- new net N$32: GTX45R.P3251_2
- new net N1A_W: GMA-245.J2401_17, GTN650.P1004_16
- new net N1A_WB: GMA-245.J2401_18, GTN650.P1004_17
- new net PT2_W: PITCH_TRIM.WHITE_GREEN
- new net PT2_WB: PITCH_TRIM.WHITE_BLUE
- new net PT2_WO: PITCH_TRIM.WHITE_ORANGE
- new net PT_W: PITCH.TRIM_IN1, PITCH.TRIM_OUT2, PITCH_TRIM.MOTOR1
- new net PT_WB: PITCH.TRIM_IN2, PITCH.TRIM_OUT1, PITCH_TRIM.MOTOR2
- new net T2_W: GTX45R.P3251_30, MFD.41_RS-232-OUT5
- new net T2_WB: GTX45R.P3251_51, MFD.37_SIGNAL_GROUND5
- new net T2_WO: GTX45R.P3251_8, MFD.24_RS-232-IN5
- new net T3_W: GSU25_PRIMARY.RS232_TX3_9, GTX45R.P3251_31
- new net T3_W0: GSU25_PRIMARY.RS232_RX3_10, GTX45R.P3251_9
- new net T3_WB: GSU25_PRIMARY.GND3_11, GTX45R.P3251_52
- new net TS_W: POSI-STROBE.GND
- new net TS_WB: POSI-STROBE.POSITION
- new net TS_WO: POSI-STROBE.STROBE
- net AUX_GTX_45R: now also GTX45R.P3251_42; no longer GTX45R.P3251_61, GTX45R.P3251_62
- net CAN_HI_W: now also GAD29.J291_1, GMA-245.J2401_36, MFD.1_CAN_BUS_HI, PITCH.CAN-H, YAW.CAN-H
- net CAN_LO_WB: now also GAD29.J291_2, GMA-245.J2401_37, MFD.2_CAN_BUS_LO, PITCH.CAN-L, YAW.CAN-L
- net PFD_37_WB: now also GTX45R.P3251_50
- net VPX_GTX_45R: no longer GTX45R.P3251_42
- net VPX_SERIAL_W: now also MFD.29_RS-232-IN3
- net VPX_SERIAL_WB: now also MFD.35_SIGNAL_GROUND3
- net VPX_SERIAL_WO: now also MFD.13_RS-232-OUT3
Other:
- moved on the sheet: ANT-ELT, GTN650, PITOT_HEAT, POSI-STROBE
