File: N_5412K.sch (EAGLE design)
At the start: 83 parts

Commit message: updating per what I wired
Parts:
- removed SW_NAV_C: (no value), switch-omron:31-XX
- removed U$9: GMC307, EAA:GMC307
- added COIL_15, IGN1_5, IGN2_5: BREAKER, EAA:BREAKER
- added D1, D2: (no value), diode:SCHOTTKY-DIODEAG
- added U$14: GMC507, EAA:GMC507
Connections:
- net ACK_GPS_RX renamed ELT_W
- net AUX_ELT renamed ELT_WO
- net GND_ELT renamed ELT_WB
- removed net GMC_307_IN1_WHT/BLU: MFD.48_RS-232-OUT1, U$9.RS-232_RX1(2)
- removed net GMC_307_OUT1_WHT: MFD.47_RS-232-IN1, U$9.RS-232_TX1(1)
- removed net GND_GMC307_GND1: U$9.POWER_GND1(5)
- removed net MASTER_ALT_SEL: ALT_SEL.P, ALT_SEL.P1, MASTER.S1
- removed net N$29: GTX45R.P3251_45
- removed net N$30: GTX45R.P3251_44
- removed net N$32: GTX45R.P3251_2
- removed net ROLL_RS232_RX_WHT: U$9.RS-232_TX2(3)
- removed net ROLL_RS232_TX_WHT/BLU: U$9.RS-232_RX2(4)
- removed net SW_WIGWAG: SW_STROBE_C.S1, U$1.J2_11
- removed net VCC: U$13.L$3
- new net E-BUSS: COIL_15.I, D1.C, D2.C, IGN1_5.I, IGN2_5.I
- new net ELT_REMOTE: U$7.REMOTE
- new net GND_KEYSWITCH: STARTER_SWITCH.GND
- new net N$27: IGN2_5.0, SYSTEM_32_2.ECU_PWR
- new net N$28: IGN1_5.0, SYSTEM_32_1.ECU_PWR
- new net SW_ALT_EN: MASTER.O1
- net AUX_CONTACTOR: now also AVIONICS.P; no longer AVIONICS.S
- net AUX_GMC_307: now also U$14.AIRCRAFT_POWER_2(9); no longer U$9.AIRCRAFT_POWER_2(9)
- net AUX_GTX_45R: now also AUX_FUSEBLOCK.20, GTX45R.P3251_61, GTX45R.P3251_62; no longer GTX45R.P3251_42
- net AUX_SENSORS: now also U$3.P$2; no longer OIL_SWITCH.P$1
- net BATT_AUX: now also D2.A
- net CAN_HI_W: now also GAD29.CAN_HI_1, GTR-20.CAN_HI_7, U$14.CAN_HI(3); no longer GAD29.J291_1, GMA-245.J2401_36, GTR-20.J2001_7
- net CAN_LO_WB: now also GAD29.CAN_LO_2, GTR-20.CAN_LO_6, U$14.CAN_LO(4); no longer GAD29.J291_2, GTR-20.J2001_6
- net GND: now also AVIONICS.O, MASTER.O; no longer AVIONICS.P, MASTER.P
- net GND_GMC307_GND2: now also U$14.POWER_GND2(15); no longer U$9.POWER_GND2(15)
- net GND_HOBBS: now also OIL_SWITCH.P$1; no longer U$3.P$2
- net LEFT_IGN_P_LEAD: now also SYSTEM_32_2.P-LEAD
- net MAIN_BUS(2GA): now also D1.A
- net MAIN_CONTACTOR: now also MASTER.P; no longer MASTER.S
- net N$31: now also COIL_15.0, SYSTEM_32_1.IGN_PWR, SYSTEM_32_2.IGN_PWR; no longer GTX45R.P3251_24
- net RIGHT_IGN_P_LEAD: now also SYSTEM_32_1.P-LEAD
- net SEN_HOBBS: now also U$3.P$1
- net SW_ALT1: now also ALT_SEL.O1; no longer ALT_SEL.O
- net SW_ALT2: now also ALT_SEL.O, U$1.J2_8; no longer ALT_SEL.O1, U$1.J2_10
- net SW_AVIONICS_MASTER: now also AVIONICS.O1; no longer AVIONICS.S1
- net SW_NAV: now also SW_STROBE_C.S; no longer SW_NAV_C.S
- net SW_STROBE: now also SW_STROBE_C.O1, U$1.J2_10; no longer SW_STROBE_C.S, U$1.J2_8
- net VPX_GMC_307: now also U$14.AIRCRAFT_POWER1(7); no longer U$9.AIRCRAFT_POWER1(7)
- net VPX_GTX_45R: now also GTX45R.P3251_42
Other:
- note added: "Done"
- note added: "Power-Deuce-Schottky"

Commit message: Cleaning ground and autopilot wiring paths
Parts:
- added SW_AUTOPILOT_DISC: (no value), switch-omron:31-XX
Connections:
- net VPX_LIGHT_NAV renamed N$38
- removed net RTRIM1_W/G: U$13.P$12
- removed net RTRIM2_W/G: U$13.P$11
- new net GND_AUTOPILOT_ROLL: U$13.P$9
- new net N$29: ROLL.TRIM_OUT1, ROLL_TRIM.MOTOR2
- new net N$30: ROLL.TRIM_OUT2, ROLL_TRIM.MOTOR1
- new net N$32: ROLL_TRIM.WHITE_BLUE, U$13.L$6
- net CWS_DISC_WB: now also SW_AUTOPILOT_DISC.P, U$13.P$15
- net GND_GEA24_1_B: no longer U$12.P$20
- net GND_GEA24_2_B: no longer U$12.P$10
- net N$14: now also ROLL_TRIM.WHITE_GREEN, U$13.L$8; no longer ROLL.TRIM_OUT1, U$13.L$13
- net N$15: now also ROLL_TRIM.WHITE_ORANGE, U$13.L$7; no longer ROLL.TRIM_OUT2, U$13.L$14
- net PITCH_WHT1: now also U$13.P$11
- net PITCH_WHT2: now also U$13.P$12
- net ROLL_WHT/BLU: now also U$13.P$6
- net ROLL_WHT/GRN: now also U$13.P$8
- net ROLL_WHT/ORN: now also U$13.P$7
- net VPX_GSA_28_2: now also U$13.P$10
Other:
- moved on the sheet: ROLL_TRIM
